File: electric/digirig-mobile-panelsx48.kicad_pcb (KiCad board)
At the start: 2 copper layers, 204 x 261 mm, 4 parts

Commit message: Digirig 1.8
- Moved attenuator on the other side of decoupling capacitor
- Changed attenuator's ratio
- Added low pass filter on audio input to suppress RF
Parts:
- moved REF** 1.60 mm to (197.4, 251.0)
- moved REF** 1.60 mm to (197.4, 15.0)
Other:
- board size 204 x 261 mm -> 202.4 x 261 mm
